File: PCB/battery_pack/18650/18650_pack_v1.sch (EAGLE design)
At the start: 6 parts, among them P1 39-30-02, X1 5566-2, X2 5566-2

Commit message: added README.md, CAMOutputes, parts_list.txt, and BOM*.csv files for the 18650 battery pack
Other:
- note added: "18650 LiPo Clips"
- note added: "Power Out"
Changed lines of the file:
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@@
 <part name="P1" library="con-molex-mini-fit" deviceset="39-30-?02?" device=""/>
 <part name="X2" library="con-molex" library_urn="urn:adsk.eagle:library:165" deviceset="5566-2" device="" package3d_urn="urn:adsk.eagle:package:8078583/1"/>
+<part name="FRAME2" library="frames" library_urn="urn:adsk.eagle:library:229" deviceset="DINA5_L" device=""/>
 </parts>
 <sheets>
 <sheet>
 <plain>
+<text x="2.54" y="78.74" size="3.81" layer="94">18650 LiPo Clips</text>
+<text x="-53.34" y="58.42" size="3.81" layer="94">Power Out</text>
 </plain>
 <instances>
@@
 <attribute name="VALUE" x="-44.958" y="51.943" size="1.778" layer="96" rot="R180"/>
 </instance>
+<instance part="FRAME2" gate="G$1" x="-99.06" y="-38.1" smashed="yes">
+<attribute name="DRAWING_NAME" x="41.91" y="-22.86" size="2.54" layer="94"/>
+<attribute name="LAST_DATE_TIME" x="41.91" y="-27.94" size="2.286" layer="94"/>
+<attribute name="SHEET" x="55.245" y="-33.02" size="2.54" layer="94"/>
+</instance>
 </instances>
