File: PCB/mainboard/small_pcb/explorator_mainboard_v2_58mm_B.sch (EAGLE design)
At the start: 58 parts, among them CN1 0.1uf, CN10 0.1uf, CN2 0.1uf, CN3 0.1uf, CN4 0.1uf, CN5 0.1uf, CN6 0.1uf, CN7 0.1uf, CN8 0.1uf, CN9 0.1uf, M1 5566-2, P1 B10B-PH-K, P2 B4B-PH-K, Q1 PNO8L07, Q2 PNO8L07, U2 SHTC3

Commit message: updated the mainboard's with the new information found in other folders including net_lists, parts_lists, pin_lists, and such
Parts:
- removed CN1, CN10, CN2, CN3, CN4, CN5, CN6, CN7, CN8, CN9: 0.1uf, resistor:C-USC0805K
- removed NEO1, NEO10, NEO2, NEO3, NEO4, NEO5, NEO6, NEO7, NEO8, NEO9: WS2812B5050, nathans-custom-parts:WS2812B5050
- removed R5: 300 R, audio amplifier example:R-US_R0805
- added CN11, CN12, CN13, CN14, CN15, CN16, CN17, CN18, CN19, CN20: 0.1uf, resistor:C-USC0805K
- added JP2: JUMPER-SMT_3_1-NC_TRACE_SILK, SparkFun-Jumpers:JUMPER-SMT_3_1-NC_TRACE_SILK
- added NEO11, NEO12, NEO13, NEO14, NEO15, NEO16, NEO17, NEO18, NEO19, NEO20: WS2812B5050, nathans-custom-parts:WS2812B5050
- added R2: 300 R, audio amplifier example:R-US_R0805
Connections:
- removed net INT: VMEL1.INT, VMEL2.INT
- removed net N$1 (its old number): NEO4.DO, NEO5.DI
- removed net N$11: NEO8.DO, NEO9.DI
- removed net N$12: NEO10.DI, NEO9.DO
- removed net N$15: NEO10.DO, NEO6.DI
- removed net N$16: NEO6.DO, NEO7.DI
- removed net N$2 (its old number): NEO1.DI, NEO5.DO
- removed net N$4: NEO1.DO, NEO2.DI
- removed net N$5: NEO2.DO, NEO3.DI
- removed net N$6: NEO3.DO, NEO8.DI
- removed net N$8: NEO4.DI, R5.1
- removed net NOUT: P1.4
- new net N$17: NEO14.DO, NEO15.DI
- new net N$18: NEO12.DI, NEO15.DO
- new net N$19: NEO11.DI, NEO12.DO
- new net N$20: NEO11.DO, NEO13.DI
- new net N$21: NEO13.DO, NEO18.DI
- new net N$22: NEO14.DI, R2.1
- new net N$23: NEO18.DO, NEO19.DI
- new net N$26: NEO19.DO, NEO20.DI
- new net N$27: NEO16.DI, NEO20.DO
- new net N$28: NEO16.DO, NEO17.DI
- new net NOUT_01: JP2.2, P1.4
- new net VEML_INT1: U$1.2, VMEL1.INT
- new net VEML_INT2: U$1.1/TX1/T, VMEL2.INT
- net 5V: now also CN11.1, CN12.1, CN13.1, CN14.1, CN15.1, CN16.1, CN17.1, CN18.1, CN19.1, CN20.1, NEO11.VDD, NEO12.VDD, NEO13.VDD, NEO14.VDD, NEO15.VDD, NEO16.VDD, NEO17.VDD, NEO18.VDD, NEO19.VDD, NEO20.VDD; no longer CN1.1, CN10.1, CN2.1, CN3.1, CN4.1, CN5.1, CN6.1, CN7.1, CN8.1, CN9.1, NEO1.VDD, NEO10.VDD, NEO2.VDD, NEO3.VDD, NEO4.VDD, NEO5.VDD, NEO6.VDD, NEO7.VDD, NEO8.VDD, NEO9.VDD
- net GND: now also CN11.2, CN12.2, CN13.2, CN14.2, CN15.2, CN16.2, CN17.2, CN18.2, CN19.2, CN20.2, NEO11.GND, NEO12.GND, NEO13.GND, NEO14.GND, NEO15.GND, NEO16.GND, NEO17.GND, NEO18.GND, NEO19.GND, NEO20.GND; no longer CN1.2, CN10.2, CN2.2, CN3.2, CN4.2, CN5.2, CN6.2, CN7.2, CN8.2, CN9.2, NEO1.GND, NEO10.GND, NEO2.GND, NEO3.GND, NEO4.GND, NEO5.GND, NEO6.GND, NEO7.GND, NEO8.GND, NEO9.GND
- net NEO1_OUT: now also NEO17.DO; no longer NEO7.DO
- net NEO_OUT: now also JP2.3
- net NEO_PIX1: now also R2.2; no longer R5.2
- net NEO_PIX2: now also JP2.1; no longer P1.5
Other:
- note added: "Ambient Light Sensing"
- note added: "Connectors"
- note added: "NeoPixel LEDs"
- note added: "NeoPixels"
- note added: "Solenoid and Motor Control"
- note added: "Temp/Humid Sensor"
- note removed: "Add decoupling caps for teensy"
- note removed: "LDRs are not connected!!!!!!"
- note removed: "Make sure this cap is placed with correct polarity"
- note removed: "Neo Pixels"
- note removed: "Neo2 is for external neopixels"
- note removed: "NeoP1 is for the onboard neo's"
- note removed: "Perhaps replace the JST ph connectors for the microphone boards to the onboard footprints"
- note removed: "Solenoids and Motors"
- note removed: "TODO - add jumper which allows for neop connector to switch between Neo1 and Neo2"
- note removed: "add fault for the motor driver"
- note removed: "make a single connector to the eye-stock"
